File: hardware/vehicle-can-collector/vehicle-can-collector.kicad_pcb (KiCad board)
At the start: 2 copper layers, 211 parts, among them J301 Micro_SD_Card_Det, J302 USB_B_Micro, J303 I2C_STANDARD, J401 OBDII Connector, Q501 DMG2301L, Q502 MMBT3906, Q503 DMG2301L, Q504 DMG2301L, Q505 DMG2301L, Q506 2N7002, Q507 DMG2301L, Q508 2N7002, Q701 2N7002, Q702 2N7002, Q703 2N7002, Q704 2N7002, Q705 2N7002, Q706 2N7002, Q707 2N7002, Q801 2N7002, Q802 2N7002, Q803 DMG2301L, Q804 2N7002, Q805 2N7002, Q806 2N7002, Q807 2N7002, Q901 2N7002, Q902 2N7002, Q903 2N7002, Q904 MMBT3904, SW201 SW_Push, U1101 TCA9534, U201 ATSAMC21J18A-AUT, U202 PL133-37TI, U203 ADM6320BX33ARJZ-R7, U301 FT2232HL, U302 93C56B, U501 LMZ12001TZX-ADJ_NOPB, U502 LM317L_SOT-89, U503 LP38693MP-3.3, U601 NCS20072, U701 MCP2557FD-xMF, U702 MCP2557FD-xMF, U703 MCP2515-xST, U704 TCA9534, U705 TH8056KDC-AAA-008-RE, U801 NCS20072, U901 NCS20072, X201 ASV-12.000MHZ-EJ-T

Commit message: Started laying out PCB
Parts:
- C510, D401, D402, D403, D404, D405: moved to B.Cu
- moved C1001 278.8 mm to (414.2, 145.6)
- moved C1003 278.8 mm to (423.9, 136.6)
- moved C1004 278.8 mm to (414.2, 142.6)
- moved C1005 278.8 mm to (419.0, 142.6)
- moved C1008 278.8 mm to (419.0, 136.6)
- moved C1011 278.8 mm to (419.0, 139.6)
- moved C1012 278.8 mm to (414.2, 136.6)
- moved C1014 278.8 mm to (414.2, 139.6)
- moved C301 278.8 mm to (385.1, 130.0)
- moved C702 278.8 mm to (337.8, 125.3)
- moved C705 278.8 mm to (359.9, 107.2)
- moved D1102 278.8 mm to (382.1, 140.5)
- moved D1106 278.8 mm to (373.3, 153.2)
- moved D1107 278.8 mm to (382.1, 143.5)
- moved D1110 278.8 mm to (373.3, 147.1)
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Routing:
- net GND: track 0.00 -> 73.0 mm, vias 0 -> 29
- net +5V_SW: track 0.00 -> 49.4 mm, vias 0 -> 5
- net +12V: track 0.00 -> 36.6 mm
- net +3V3: track 0.00 -> 34.3 mm, vias 0 -> 10
- net +5V: track 0.00 -> 30.9 mm, vias 0 -> 7
- net HS_CAN_LO: track 0.00 -> 25.2 mm
- net Net-(D501-Pad1): track 0.00 -> 21.4 mm
- net ~{PWR_CTRL}: track 0.00 -> 18.3 mm, vias 0 -> 2
- net HS_CAN_HI: track 0.00 -> 16.0 mm, vias 0 -> 1
- net Net-(C505-Pad1): track 0.00 -> 15.5 mm
- net Net-(Q503-Pad1): track 0.00 -> 13.8 mm
- net +12V_SW: track 0.00 -> 12.7 mm
- net V_J1850: track 0.00 -> 11.0 mm
- net Net-(C504-Pad2): track 0.00 -> 8.78 mm
- net Net-(C503-Pad2): track 0.00 -> 8.69 mm
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- added copper zone on In2.Cu, net +3V3
- added copper zone on In1.Cu, net +5V
- added copper zone on B.Cu, net GND
Other:
- board outline added: 167 x 102.2 mm
- copper layers 2 -> 4

Commit message: Actually hook up CAN busses
- this required another pin shift.  DTS update to follow
Parts:
- C1001, C1002, C1003, C1004, C513, C514, C708, L501, R721: moved to B.Cu
- moved C1003 362.0 mm to (69.2, 64.1), turned to -90 degrees
- moved C1002 352.1 mm to (69.2, 57.8), turned to -90 degrees
- moved C1006 350.3 mm to (76.1, 31.9)
- moved C1007 350.3 mm to (76.1, 28.9)
- moved C1008 350.3 mm to (85.7, 28.9)
- moved C1010 350.3 mm to (76.1, 34.9)
- moved C1011 350.3 mm to (85.7, 31.9)
- moved C1012 350.3 mm to (80.9, 28.9)
- moved C1013 350.3 mm to (76.1, 37.9)
- moved C1014 350.3 mm to (80.9, 31.9)
- moved C1001 349.0 mm to (76.8, 56.5)
- moved C1004 348.8 mm to (73.7, 67.3)
- moved C1005 346.7 mm to (90.5, 31.9)
- moved R719 344.1 mm to (24.8, 56.5)
- moved C1009 343.1 mm to (85.7, 37.9)
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Connections:
- Q706 pad 3: ~{MS_CAN_EN}_5V -> ~{MS_CAN_EN_5V}
- R716 pad 2: ~{MS_CAN_EN}_5V -> ~{MS_CAN_EN_5V}
- U201 pad 1: unconnected-(U201-Pad1) -> ~{ISO_TX}
- U201 pad 2: unconnected-(U201-Pad2) -> ~{ISO_RX}
- U201 pad 23: SW_CAN_CS -> ~{HS_CAN_EN}
- U201 pad 24: SW_CAN_MISO -> ~{PWR_CTRL}
- U201 pad 27: ~{HS_CAN_EN} -> MS_CAN_TX
- U201 pad 28: ~{PWR_CTRL} -> MS_CAN_RX
- U201 pad 32: unconnected-(U201-Pad32) -> SW_CAN_LOAD
- U201 pad 35: ~{ISO_TX} -> SDCARD_MOSI
- U201 pad 36: unconnected-(U201-Pad36) -> SDCARD_SCK
- U201 pad 37: ~{ISO_RX} -> SW_CAN_CS
- U201 pad 38: SW_CAN_LOAD -> SW_CAN_MISO
- U201 pad 43: SDCARD_MOSI -> HS_CAN_TX
- U201 pad 44: SDCARD_SCK -> HS_CAN_RX
Routing:
- net +12V_SW: track 12.7 -> 113.0 mm, vias 0 -> 2
- net +3V3_SW: track 4.06 -> 85.9 mm, vias 0 -> 4
- net SW_CAN_MODE1: track 0.00 -> 78.9 mm, vias 0 -> 5
- net ~{HS_CAN_EN}: track 1.60 -> 79.4 mm, vias 0 -> 6
- net SW_CAN_MODE0: track 0.00 -> 77.1 mm, vias 0 -> 5
- net ~{PWR_CTRL}: track 18.3 -> 78.8 mm, vias 2 -> 5
- net ~{MS_CAN_EN}: track 0.00 -> 60.0 mm, vias 0 -> 6
- net SW_CAN_CS: track 0.00 -> 57.1 mm, vias 0 -> 5
- net SW_CAN_MISO: track 0.00 -> 55.7 mm, vias 0 -> 5
- net HS_CAN_TX: track 1.87 -> 54.8 mm, vias 0 -> 5
- net SW_CAN_LOAD: track 0.00 -> 46.8 mm, vias 0 -> 4
- net CLK_CAN: track 0.00 -> 46.3 mm, vias 0 -> 3
- net MS_CAN_RX: track 0.00 -> 44.0 mm, vias 0 -> 4
- net +3V3: track 34.3 -> 77.4 mm, vias 10 -> 22
- net SW_CAN_SCK: track 0.00 -> 41.4 mm, vias 0 -> 3
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
Commit message: Finished first round of layout.
- dang this has a lot of parts!
Parts:
- added J304: M04JST, SparkFun-Connectors:1X04-1.5MM_JST, F.Cu at (141.9, 47.9)
- added REF**: OSHW-Logo2_14.6x12mm_SilkScreen, Symbol:OSHW-Logo2_14.6x12mm_SilkScreen, F.Cu at (151.8, 126.4)
- C1005, C1006, C1007, C1008, C1009, C1010, C1011, C1012, C1013, C1014, C201, C602, C801, Q901, R1101, R1102, R1103, R1104, R1105, R303, R902, R903, R904, R905, R906, R908, R909: moved to B.Cu
- moved R602 376.7 mm to (89.5, 116.2), turned to -90 degrees
- moved R601 375.3 mm to (87.0, 116.2), turned to 90 degrees
- moved D805 375.2 mm to (93.3, 135.3)
- moved R815 372.5 mm to (87.6, 137.2)
- moved D803 370.5 mm to (87.9, 128.3)
- moved R806 370.3 mm to (97.2, 126.6), turned to 90 degrees
- moved C801 367.5 mm to (94.0, 130.2), turned to -90 degrees
- moved R809 366.8 mm to (95.5, 123.2)
- moved R808 366.6 mm to (87.6, 130.8), turned to 180 degrees
- moved Q904 364.6 mm to (75.6, 112.4), turned to 90 degrees
- moved D601 363.4 mm to (92.1, 111.8), turned to 90 degrees
- moved C602 361.6 mm to (95.9, 114.9)
- moved R807 361.4 mm to (91.4, 123.2)
- moved R907 360.9 mm to (75.6, 115.6)
- moved C601 360.6 mm to (92.1, 116.2), turned to -90 degrees
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Connections:
- U201 pad 23: ~{HS_CAN_EN} -> unconnected-(U201-Pad23)
- U201 pad 25: unconnected-(U201-Pad25) -> ~{HS_CAN_EN}
- U201 pad 32: SW_CAN_LOAD -> unconnected-(U201-Pad32)
- U201 pad 35: SDCARD_MOSI -> unconnected-(U201-Pad35)
- U201 pad 36: SDCARD_SCK -> SW_CAN_LOAD
- U201 pad 43: HS_CAN_TX -> SDCARD_MOSI
- U201 pad 44: HS_CAN_RX -> SDCARD_SCK
- U201 pad 49: SW_CAN_MODE0 -> HS_CAN_TX
- U201 pad 5: unconnected-(U201-Pad5) -> SW_CAN_MODE0
- U201 pad 50: SW_CAN_MODE1 -> HS_CAN_RX
- U201 pad 6: unconnected-(U201-Pad6) -> SW_CAN_MODE1
- U301 pad 16: OUTPUT_RX -> ~{OUTPUT_RX}
- U301 pad 17: OUTPUT_TX -> ~{OUTPUT_TX}
Routing:
- net GND: track 104.6 -> 243.9 mm, vias 46 -> 80
- net J1850_BUS+: track 3.12 -> 139.0 mm, vias 0 -> 3
- net SAE_PWM: track 2.32 -> 122.6 mm, vias 0 -> 7
- net J1850_BUS-: track 3.28 -> 118.7 mm, vias 0 -> 3
- net BAT_LEVEL: track 0.00 -> 107.5 mm, vias 0 -> 7
- net ~{ISO_TX}: track 0.00 -> 90.6 mm, vias 0 -> 8
- net J1850_TX+: track 0.00 -> 85.7 mm, vias 0 -> 5
- net J1850_RX: track 0.00 -> 85.6 mm, vias 0 -> 7
- net ~{ISO_RX}: track 0.00 -> 83.4 mm, vias 0 -> 8
- net SAE_LEVEL: track 0.00 -> 80.8 mm, vias 0 -> 6
- net +3V3: track 77.4 -> 158.1 mm, vias 22 -> 48
- net ISO_K: track 0.00 -> 76.7 mm, vias 0 -> 5
- net J1850_TX-: track 0.00 -> 73.7 mm, vias 0 -> 6
- net VBUS: track 0.00 -> 67.4 mm, vias 0 -> 2
- net SDA: track 19.7 -> 77.1 mm, vias 0 -> 5
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- added copper zone on In1.Cu, net +1V8
Other:
- board size 167 x 102.2 mm -> 102.2 x 102.9 mm
- board text added: "(c) 2022 Gavin Hurlbut"
- board text added: "Vehicle CAN Collector v1"

Commit message: Finished rebasing, and then fix PCB and generate gerbers
Routing:
- net K_LINE: track 6.85 -> 24.2 mm, vias 0 -> 1
- net MS_CAN_HI: track 5.88 -> 17.1 mm, vias 0 -> 1
- net HS_CAN_HI: track 6.35 -> 16.5 mm, vias 0 -> 1
- net GND: track 243.9 -> 250.8 mm, vias 80 -> 81
- net ISO_K: track 76.7 -> 77.5 mm, vias 5 -> 6
- net HS_CAN_TX: track 53.1 -> 52.4 mm
- net J1850_TX+: vias 5 -> 7
- net J1850_RX: vias 7 -> 8
